File: PCB/TesterV1/2.kicad_sch (KiCad schematic)
At the start: 11 parts, among them J1 Connector, USB-TYPE-C-16P, U3 ESP32-WROOM-32E, U4 AMS1117-3.3, U5 CH340C

Commit message: Update PCB footprints, nets and ignore PCB/
Add .gitignore to exclude PCB/ and apply multiple PCB library updates: rename nets (e.g. VCC->BAT, CHRG, STDBY), reassign nets on several pads, and update schematic and fp-info-cache. Replace/update footprints and metadata: convert several resistor footprints from 0402 to 0805 (adjusting values, sizes, pads and 3D models), change fuse footprint to a tactile switch footprint, and update datasheets, LCSC IDs, stock and price fields. Adjust pad geometry, silk/fab text positions/rotations and various UUIDs to match the new footprints and orientation changes.
Parts:
- added BT1: Battery Holder, Battery:BatteryHolder_MPD_BH-18650-PC2, symbol Device:Battery_Cell
- added C1: 10uF, PCM_JLCPCB:C_0603, symbol PCM_JLCPCB-Capacitors:0603,10uF
- added D1: Green, PCM_JLCPCB:D_0805, symbol PCM_JLCPCB-Diodes:LED,0805,Green
- added D2: Red, PCM_JLCPCB:D_0805, symbol PCM_JLCPCB-Diodes:LED,0805,Red
- added J2: XLR3, Connector_Audio:Jack_XLR_Neutrik_NC3FAAH-0_Horizontal, symbol Connector_Audio:XLR3
- added R3, R4: 1kΩ, PCM_JLCPCB:R_0402, symbol PCM_JLCPCB-Resistors:0402,1kΩ
- added R7: 1.5kΩ, PCM_JLCPCB:R_0402, symbol PCM_JLCPCB-Resistors:0402,1.5kΩ
- added U1: TP4057, PCM_JLCPCB:SOT-23-6_L2.9-W1.6-P0.95-LS2.8-BL, symbol PCM_JLCPCB-Power:Battery, Li-Ion, 0.5A, TP4057
Connections:
- net GND: now also BT1.2 (-), C1.2, R7.2, U1.2 (GND)
- net VCC renamed +5V
- net +5V: now also R3.1, R4.1, U1.4 (VCC)
- new net: D2.2, R4.2
- new net: R7.1, U1.6 (PROG)
- new net: D1.2, R3.2
- new net BAT: BT1.1 (+), C1.1, U1.3 (BAT)
- new net CHRG: D1.1, U1.1 (CHRG)
- new net STDBY: D2.1, U1.5 (STDBY)
- no-connect marks 0 -> 9
Other:
- note added: "Battery"
- note added: "Cell"
- note added: "Charging IC"
- note added: "Led indication"

Commit message: Update 2.kicad_sch
Parts:
- added J3: XLR3, Connector_Audio:Jack_XLR_Neutrik_NC3FAAH-0_Horizontal, symbol Connector_Audio:XLR3
Changed lines of the file:
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@@
+	)
+	(symbol
+		(lib_id "Connector_Audio:XLR3")
+		(at 181.61 121.92 0)
+		(unit 1)
+		(exclude_from_sim no)
+		(in_bom yes)
+		(on_board yes)
+		(dnp no)
+		(fields_autoplaced yes)
+		(property "Reference" "J3"
+			(at 181.61 111.76 0)
+			(effects
+				(font
+					(size 1.27 1.27)
+				)
+			)
+		)
+		(property "Value" "XLR3"
+			(at 181.61 114.3 0)
+			(effects
+				(font
+					(size 1.27 1.27)
+				)
+			)
+		)
+		(property "Footprint" "Connector_Audio:Jack_XLR_Neutrik_NC3FAAH-0_Horizontal"
+			(at 181.61 121.92 0)
+			(effects
+				(font
+					(size 1.27 1.27)
+				)
+				(hide yes)
+			)
+		)
+		(property "Datasheet" "~"
+			(at 181.61 121.92 0)
+			(effects
+				(font
+					(size 1.27 1.27)
+				)
+				(hide yes)
+			)
+		)
+		(property "Description" "XLR Connector, Male or Female, 3 Pins"
+			(at 181.61 121.92 0)
+			(effects
+				(font
+					(size 1.27 1.27)
+				)
+				(hide yes)
+			)
+		)
+		(pin "3"
+		)
+		(pin "2"
+		)
+		(pin "1"
+		)
+		(instances
+			(project "2"
+				(path "/110d0971-d5ef-41f2-b31e-1420793f002b"
+					(reference "J3")
+					(unit 1)
+				)
+			)
+		)
 	)
 	(symbol
